File: PCB/Hackpad.kicad_sch (KiCad schematic)
At the start: 8 parts, among them SW1 SW_Push, SW2 SW_Push, SW3 SW_Push, SW4 SW_Push, SW6 RotaryEncoder, U1 XIAO-RP2040-DIP

Commit message: Add files via upload
Parts:
- D1, D2: footprint LED_SMD:LED_SK6812MINI_PLCC4_3.5x3.5mm_P1.75mm -> Hackclub Footprints:MX_SK6812MINI-E_REV
- U1: footprint OPL Lib:XIAO-RP2040-DIP -> Hackclub Footprints:XIAO-RP2040-DIP
